File: ergogen-output/pcbs/final-left.kicad_pcb (KiCad board)
At the start: 2 copper layers, 161.7 x 120.6 mm, 61 parts

Commit message: fix pcbs :(
Routing:
- net P009: track 160.8 -> 164.2 mm
- net pos: track 160.9 -> 162.9 mm
Changed lines of the file:
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@@
 	)
 	(segment
-		(start 88.955604 70.22)
-		(end 121.447306 70.22)
+		(start 146.26 80.23)
+		(end 140.0525 74.0225)
 		(width 0.25)
 		(layer "B.Cu")
@@
 	)
 	(segment
-		(start 140.0525 74.0225)
-		(end 146.26 80.23)
+		(start 61.7315 84.5725)
+		(end 57.085 89.219)
 		(width 0.25)
 		(layer "B.Cu")
@@
 	)
 	(segment
-		(start 121.447306 70.22)
-		(end 125.249806 74.0225)
+		(start 74.603104 84.5725)
+		(end 61.7315 84.5725)
 		(width 0.25)
 		(layer "B.Cu")
@@
 	)
 	(segment
-		(start 57.085 92.39)
-		(end 57.085 112.44)
+		(start 88.563604 70.612)
+		(end 74.603104 84.5725)
 		(width 0.25)
 		(layer "B.Cu")
@@
 	)
 	(segment
-		(start 57.085 112.44)
-		(end 57.085 132.49)
+		(start 123.8065 74.0225)
+		(end 120.396 70.612)
 		(width 0.25)
 		(layer "B.Cu")
@@
 	)
 	(segment
-		(start 68.279 78.025)
-		(end 81.150604 78.025)
+		(start 120.396 70.612)
+		(end 88.563604 70.612)
 		(width 0.25)
 		(layer "B.Cu")
@@
 	(segment
 		(start 57.085 92.39)
-		(end 57.085 89.219)
+		(end 57.085 112.44)
 		(width 0.25)
 		(layer "B.Cu")
@@
 	(segment
 		(start 57.085 89.219)
-		(end 68.279 78.025)
+		(end 57.085 92.39)
 		(width 0.25)
 		(layer "B.Cu")
@@
 	)
 	(segment
-		(start 81.150604 78.025)
-		(end 88.955604 70.22)
+		(start 57.085 112.44)
+		(end 57.085 132.49)
 		(width 0.25)
 		(layer "B.Cu")
@@
 	)
 	(segment
-		(start 125.249806 74.0225)
-		(end 140.0525 74.0225)
+		(start 140.0525 74.0225)
+		(end 123.8065 74.0225)
 		(width 0.25)
 		(layer "B.Cu")
@@
 	)
 	(segment
+		(start 77.135 92.39)
+		(end 77.135 82.804)
+		(width 0.25)
+		(layer "B.Cu")
+		(net 6)
+	)
+	(segment
 		(start 77.135 132.49)
 		(end 77.135 152.54)
@@
 	)
 	(segment
-		(start 77.135 82.677)
-		(end 89.142 70.67)
+		(start 120.267604 71.12)
+		(end 123.620104 74.4725)
 		(width 0.25)
 		(layer "B.Cu")
@@
 	)
 	(segment
-		(start 77.135 92.39)
-		(end 77.135 82.677)
+		(start 88.819 71.12)
+		(end 120.267604 71.12)
 		(width 0.25)
 		(layer "B.Cu")
@@
 	)
 	(segment
-		(start 125.021292 74.4725)
+		(start 123.620104 74.4725)
 		(end 137.9625 74.4725)
 		(width 0.25)
@@
 	)
 	(segment
-		(start 89.142 70.67)
-		(end 121.218792 70.67)
+		(start 137.9625 74.4725)
+		(end 143.72 80.23)
 		(width 0.25)
 		(layer "B.Cu")
@@
 	)
 	(segment
-		(start 137.9625 74.4725)
-		(end 143.72 80.23)
+		(start 77.135 82.804)
+		(end 77.135 82.677)
 		(width 0.25)
 		(layer "B.Cu")
@@
 	)
 	(segment
-		(start 121.218792 70.67)
-		(end 125.021292 74.4725)
+		(start 77.135 82.804)
+		(end 88.819 71.12)
 		(width 0.25)
 		(layer "B.Cu")
@@
 	(segment
 		(start 97.185 77.677)
-		(end 103.742 71.12)
+		(end 103.2895 71.5725)
 		(width 0.25)
 		(layer "B.Cu")
@@
 	)
 	(segment
-		(start 121.032396 71.12)
-		(end 124.834896 74.9225)
+		(start 97.185 84.39)
+		(end 97.185 77.677)
 		(width 0.25)
 		(layer "B.Cu")
@@
 	)
 	(segment
-		(start 124.834896 74.9225)
-		(end 135.8725 74.9225)
+		(start 97.185 84.39)
+		(end 97.185 104.44)
 		(width 0.25)
 		(layer "B.Cu")
@@
 	)
 	(segment
-		(start 97.185 84.39)
-		(end 97.185 104.44)
+		(start 135.8725 74.9225)
+		(end 141.18 80.23)
 		(width 0.25)
 		(layer "B.Cu")
@@
 	)
 	(segment
-		(start 97.185 84.39)
-		(end 97.185 77.677)
+		(start 120.083708 71.5725)
+		(end 123.433708 74.9225)
 		(width 0.25)
 		(layer "B.Cu")
@@
 	)
 	(segment
-		(start 135.8725 74.9225)
-		(end 141.18 80.23)
+		(start 103.2895 71.5725)
+		(end 120.083708 71.5725)
 		(width 0.25)
 		(layer "B.Cu")
@@
 	)
 	(segment
-		(start 103.742 71.12)
-		(end 121.032396 71.12)
+		(start 97.185 124.49)
+		(end 97.185 144.54)
 		(width 0.25)
 		(layer "B.Cu")
@@
 	)
 	(segment
-		(start 97.185 124.49)
-		(end 97.185 144.54)
+		(start 123.433708 74.9225)
+		(end 135.8725 74.9225)
 		(width 0.25)
 		(layer "B.Cu")
@@
 	)
 	(segment
+		(start 64.34 80.44)
+		(end 65.024 79.756)
+		(width 0.2)
+		(layer "F.Cu")
+		(net 44)
+	)
+	(segment
 		(start 106.6 72.85)
 		(end 104.44 72.85)
@@
 	)
 	(segment
-		(start 72.165 78.025)
-		(end 84.215 78.025)
-		(width 0.25)
-		(layer "F.Cu")
-		(net 44)
-	)
-	(segment
 		(start 45.5675 84.5725)
 		(end 63.0625 84.5725)
@@
 	)
 	(segment
-		(start 64.34 85.85)
-		(end 72.165 78.025)
-		(width 0.25)
-		(layer "F.Cu")
-		(net 44)
-	)
-	(segment
 		(start 129.535 94.415)
 		(end 129.535 86.863)
@@
 	)
 	(segment
+		(start 65.024 79.756)
+		(end 82.484 79.756)
+		(width 0.2)
+		(layer "F.Cu")
+		(net 44)
+	)
+	(segment
 		(start 84.215 78.025)
 		(end 84.39 77.85)
@@
 	)
 	(segment
+		(start 82.484 79.756)
+		(end 84.39 77.85)
+		(width 0.2)
+		(layer "F.Cu")
+		(net 44)
+	)
+	(segment
 		(start 128.48 95.47)
 		(end 129.535 94.415)
@@
 	)
 	(segment
+		(start 64.34 85.85)
+		(end 64.34 80.44)
+		(width 0.2)
+		(layer "F.Cu")
+		(net 44)
+	)
+	(segment
 		(start 126.3459 78.5059)
 		(end 124.49 76.65)
@@
 	)
 	(segment
-		(start 114.3 122.48165)
-		(end 114.3 136.200131)
+		(start 113.3375 117.2945)
+		(end 112.085 118.547)
 		(width 0.25)
 		(layer "B.Cu")
@@
 	)
 	(segment
-		(start 110.15 108.95)
-		(end 113.3375 112.1375)
+		(start 140.716 153.924)
+		(end 150.876 164.084)
 		(width 0.25)
 		(layer "B.Cu")
@@
 	)
 	(segment
-		(start 150.84394 166.195723)
-		(end 171.244673 166.195723)
+		(start 114.3 136.200131)
+		(end 111.788066 138.712065)
 		(width 0.25)
 		(layer "B.Cu")
@@
 	)
 	(segment
-		(start 127.16835 155.4)
-		(end 140.048217 155.4)
+		(start 150.84394 166.195723)
+		(end 150.876 166.195723)
 		(width 0.25)
 		(layer "B.Cu")
@@
 	)
 	(segment
-		(start 113.3375 117.2945)
-		(end 112.085 118.547)
+		(start 150.876 164.084)
+		(end 150.876 166.195723)
 		(width 0.25)
 		(layer "B.Cu")
@@
 	)
 	(segment
-		(start 112.085 120.26665)
-		(end 114.3 122.48165)
+		(start 110.15 108.95)
+		(end 113.3375 112.1375)
 		(width 0.25)
 		(layer "B.Cu")
@@
 	)
 	(segment
-		(start 172.543959 151.809)
-		(end 172.035959 151.301)
+		(start 150.876 166.195723)
+		(end 171.244673 166.195723)
 		(width 0.25)
 		(layer "B.Cu")
@@
 	)
 	(segment
-		(start 112.085 118.547)
-		(end 112.085 120.26665)
+		(start 124.46 153.924)
+		(end 140.716 153.924)
 		(width 0.25)
 		(layer "B.Cu")
@@
 	)
 	(segment
-		(start 140.048217 155.4)
-		(end 150.84394 166.195723)
+		(start 114.3 122.48165)
+		(end 114.3 136.200131)
 		(width 0.25)
 		(layer "B.Cu")
@@
 	)
 	(segment
-		(start 172.035959 151.301)
-		(end 171.527959 151.301)
+		(start 112.085 120.26665)
+		(end 114.3 122.48165)
 		(width 0.25)
 		(layer "B.Cu")
@@
 	)
 	(segment
-		(start 114.3 136.200131)
-		(end 111.788066 138.712065)
+		(start 172.543959 151.809)
+		(end 172.035959 151.301)
 		(width 0.25)
 		(layer "B.Cu")
@@
 	(segment
 		(start 111.788066 138.712065)
-		(end 111.788066 140.019716)
+		(end 111.788066 141.252066)
+		(width 0.25)
+		(layer "B.Cu")
+		(net 48)
+	)
+	(segment
+		(start 172.035959 151.301)
+		(end 171.527959 151.301)
+		(width 0.25)
+		(layer "B.Cu")
+		(net 48)
+	)
+	(segment
+		(start 112.085 118.547)
+		(end 112.085 120.26665)
 		(width 0.25)
 		(layer "B.Cu")
@@
 	)
 	(segment
-		(start 111.788066 140.019716)
-		(end 127.16835 155.4)
+		(start 111.788066 141.252066)
+		(end 124.46 153.924)
 		(width 0.25)
 		(layer "B.Cu")

Commit message: Fix up PCB one last time
Parts:
- moved ? 1.60 mm to (118.6, 86.9)
Routing:
- net P024: track 85.2 -> 86.1 mm
Changed lines of the file:
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@@
 	(footprint "HOLE_M2_TH"
 		(layer "F.Cu")
-		(at 120.175 86.875)
+		(at 118.578619 86.868799)
 		(property "Reference" ""
 			(at 0 0 0)
@@
 	)
 	(segment
+		(start 116.153619 80.471381)
+		(end 117.235 79.39)
+		(width 0.25)
+		(layer "B.Cu")
+		(net 16)
+	)
+	(segment
+		(start 117.235 99.44)
+		(end 117.235 88.954648)
+		(width 0.25)
+		(layer "B.Cu")
+		(net 16)
+	)
+	(segment
 		(start 133.7825 75.3725)
 		(end 138.64 80.23)
@@
 	)
 	(segment
-		(start 117.235 79.39)
-		(end 121.2525 75.3725)
+		(start 116.153619 87.873267)
+		(end 116.153619 80.471381)
 		(width 0.25)
 		(layer "B.Cu")
@@
 	(segment
 		(start 117.235 79.39)
-		(end 117.235 99.44)
+		(end 121.2525 75.3725)
 		(width 0.25)
 		(layer "B.Cu")
@@
 		(width 0.25)
 		(layer "B.Cu")
+		(net 16)
+	)
+	(segment
+		(start 117.235 88.954648)
+		(end 116.153619 87.873267)
+		(width 0.25)
+		(layer "B.Cu")
